File: lab/ANS_Uebung3/ANS_Uebung3.kicad_sch (KiCad schematic)
At the start: 8 parts, among them Q1 BS170, Q2 BS170

Commit message: VCO 03.03.26
Parts:
- removed C2: {Cvar}, symbol Device:C_Variable
- removed Ib1: 1.58m, symbol Simulation_SPICE:IDC
- added Q3: NMOS, symbol Simulation_SPICE:NMOS
- added V1: 5, symbol Simulation_SPICE:VDC
- Vdd1: value 5 -> 10
Connections:
- net 0: now also Q3.3 (S), V1.2
- net at Q1.3 (S), Q2.3 (S): now also Q3.1 (D)
- new net: Q3.2 (G), V1.1
Other:
- note added: ".param L=100u C=1u R=47k"
- note removed: ".param Cvar=10n .control alterparam Cvar = 10n reset tran 1u 70m wrdata Cvar_10n.txt time v(/Vd1) write Cvar_10n.raw alterparam Cvar = 22n reset tran 1u 70m wrdata Cvar_22n.txt time v(/Vd1) write Cvar_22n.raw alterparam Cvar = 47n reset tran 1u 70m wrdata Cvar_47n.txt time v(/Vd1) write Cvar_47n.raw alterparam Cvar = 100n reset tran 1u 70m wrdata Cvar_100n.txt time v(/Vd1) write Cvar_100n.raw .en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"
- note removed: ".param L=1m C=1u R=1k Cvar=1u"
