File: lab/CC_VCO/CC_VCO.kicad_pcb (KiCad board)
At the start: 2 copper layers, 69.5 x 56 mm, 15 parts, among them Q1 BS170, Q2 BS170

Commit message: Platine aktualisiert
Parts:
- removed C2, C3: 10n, Capacitor_THT:C_Disc_D5.0mm_W2.5mm_P5.00mm
- L1, L2: value 3u -> 3,3u
Routing:
- net Net-(Q1-G): track 35.7 -> 0.22 mm
- net Net-(Q1-S): track 67.5 -> 47.7 mm
- net Net-(Q2-G): track 19.1 -> 0.22 mm
