File: kicad/FM-ELK_LC-VCO-FINAL/FM-ELK.kicad_pcb (KiCad board)
At the start: 2 copper layers, 0 parts

Commit message: Board aktualisiert und Python angepasst
Parts:
- added D1: 1SV149, Package_TO_SOT_THT:TO-92_Inline, F.Cu at (144.2, 77.0)
- added D2: 1SV149, Package_TO_SOT_THT:TO-92_Inline, F.Cu at (162.7, 76.9)
- added J2: Conn_Coaxial, Connector_Coaxial:BNC_Amphenol_031-5539_Vertical, F.Cu at (120.9, 73.1)
- added J3: Conn_Coaxial, Connector_Coaxial:BNC_Amphenol_031-5539_Vertical, F.Cu at (189.5, 81.0)
- added L2: 3.3u, Inductor_THT:L_Radial_D10.0mm_P5.00mm_Fastron_07P, F.Cu at (143.0, 68.5)
- added L3: 3.3u, Inductor_THT:L_Radial_D10.0mm_P5.00mm_Fastron_07P, F.Cu at (162.0, 68.5)
- added Q1: BS170, Package_TO_SOT_THT:TO-92_Inline, F.Cu at (163.5, 87.0)
- added Q2: BS170, Package_TO_SOT_THT:TO-92_Inline, F.Cu at (144.2, 87.9)
- added Q3: BS170, Package_TO_SOT_THT:TO-92_Inline, F.Cu at (150.5, 96.9)
- added Q4: BS170, Package_TO_SOT_THT:TO-92_Inline, F.Cu at (161.2, 96.9)
- added R4: 500k, Resistor_THT:R_Axial_DIN0207_L6.3mm_D2.5mm_P7.62mm_Horizontal, F.Cu at (147.5, 102.0)
- added Vdd1: 10.05, Connector_PinHeader_2.54mm:PinHeader_1x02_P2.54mm_Vertical, F.Cu at (144.0, 110.7)
- added Vtune1: 5.33, Connector_PinHeader_2.54mm:PinHeader_1x02_P2.54mm_Vertical, F.Cu at (167.0, 111.0)
Routing:
- net GND: track 0.00 -> 143.8 mm, vias 0 -> 1
- net Net-(D1-K): track 0.00 -> 137.6 mm
- net Net-(J2-Ext): track 0.00 -> 123.8 mm
- net Out: track 0.00 -> 76.5 mm
- net Net-(D1-A): track 0.00 -> 60.6 mm, vias 0 -> 1
- net Net-(Q1-S): track 0.00 -> 30.7 mm
- net Net-(Q3-G): track 0.00 -> 28.5 mm
