File: kicad/FM-ANS_LC-VCO-V2/LC VCO.kicad_sch (KiCad schematic)
At the start: 13 parts, among them Q1 BS170, Q2 BS170

Commit message: Aktuelle Version hochgeladen
Parts:
- L1, L2: value 3u -> 3.3u
- R1, R2: value 22k -> 10k
- R3: value 47k -> 10k
Changed lines of the file:
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@@
 			)
 		)
-		(property "Value" "47k"
+		(property "Value" "10k"
 			(at 125.73 118.11 90)
 			(show_name no)
@@
 			)
 		)
-		(property "Value" "22k"
+		(property "Value" "10k"
 			(at 138.43 102.87 90)
 			(show_name no)
@@
 			)
 		)
-		(property "Value" "22k"
+		(property "Value" "10k"
 			(at 113.03 102.87 90)
 			(show_name no)
@@
 			)
 		)
-		(property "Value" "3u"
+		(property "Value" "3.3u"
 			(at 102.87 73.6599 0)
 			(show_name no)
@@
 			)
 		)
-		(property "Value" "3u"
+		(property "Value" "3.3u"
 			(at 154.94 74.9299 0)
 			(show_name no)
