File: kicad/FM-ANS_LC-VCO-V3/FM-ELK.kicad_sch (KiCad schematic)
At the start: 13 parts, among them J2 Conn_Coaxial, J3 Conn_Coaxial, Q1 BS170, Q2 BS170, Q3 BS170, Q4 BS170

Commit message: Aktuelle Version hochgeladen
Parts:
- R4: value 500k -> 1500k
Connections:
- net GND: no longer J2.1 (In)
- net at D1.2 (A), D2.2 (A), Vtune1.1: now also J2.1 (In)
- net at J3.2 (Ext): now also J2.2 (Ext)
- net at L2.2, L3.2, R4.2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: no longer J2.2 (Ext)
Other:
- moved on the sheet: J2, J3
Changed lines of the file:
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@@
+	)
+	(junction
+		(at 114.3 77.47)
+		(diameter 0)
+		(color 0 0 0 0)
 	)
 	(junction
@@
 	)
 	(junction
-		(at 67.31 90.17)
-		(diameter 0)
-		(color 0 0 0 0)
-	)
-	(junction
 		(at 83.82 96.52)
 		(diameter 0)
@@
 	)
 	(junction
-		(at 83.82 114.3)
+		(at 128.27 88.9)
 		(diameter 0)
 		(color 0 0 0 0)
 	)
 	(junction
-		(at 71.12 80.01)
+		(at 83.82 114.3)
 		(diameter 0)
 		(color 0 0 0 0)
@@
 	(wire
 		(pts
-			(xy 133.35 97.79) (xy 133.35 96.52)
-		)
-		(stroke
-			(width 0)
-			(type default)
-		)
-	)
-	(wire
-		(pts
-			(xy 114.3 88.9) (xy 151.13 88.9)
+			(xy 114.3 88.9) (xy 128.27 88.9)
 		)
 		(stroke
@@
 	(wire
 		(pts
+			(xy 128.27 78.74) (xy 128.27 88.9)
+		)
+		(stroke
+			(width 0)
+			(type default)
+		)
+	)
+	(wire
+		(pts
 			(xy 119.38 100.33) (xy 106.68 100.33)
 		)
@@
 	(wire
 		(pts
-			(xy 71.12 80.01) (xy 74.93 80.01)
+			(xy 123.19 73.66) (xy 114.3 73.66)
+		)
+		(stroke
+			(width 0)
+			(type default)
+		)
+	)
+	(wire
+		(pts
+			(xy 67.31 80.01) (xy 74.93 80.01)
 		)
 		(stroke
@@
 	(wire
 		(pts
-			(xy 119.38 91.44) (xy 119.38 100.33)
+			(xy 119.38 92.71) (xy 119.38 100.33)
 		)
 		(stroke
@@
 	(wire
 		(pts
+			(xy 114.3 73.66) (xy 114.3 77.47)
+		)
+		(stroke
+			(width 0)
+			(type default)
+		)
+	)
+	(wire
+		(pts
 			(xy 83.82 90.17) (xy 83.82 96.52)
 		)
@@
 	(wire
 		(pts
-			(xy 54.61 90.17) (xy 67.31 90.17)
-		)
-		(stroke
-			(width 0)
-			(type default)
-		)
-	)
-	(wire
-		(pts
 			(xy 83.82 96.52) (xy 83.82 101.6)
 		)
@@
 	(wire
 		(pts
-			(xy 67.31 80.01) (xy 71.12 80.01)
-		)
-		(stroke
-			(width 0)
-			(type default)
-		)
-	)
-	(wire
-		(pts
 			(xy 95.25 107.95) (xy 95.25 101.6)
 		)
@@
 	(wire
 		(pts
-			(xy 59.69 74.93) (xy 71.12 74.93)
-		)
-		(stroke
-			(width 0)
-			(type default)
-		)
-	)
-	(wire
-		(pts
 			(xy 83.82 101.6) (xy 95.25 101.6)
 		)
@@
 	(wire
 		(pts
-			(xy 151.13 97.79) (xy 133.35 97.79)
+			(xy 151.13 97.79) (xy 128.27 97.79)
 		)
 		(stroke
@@
 	(wire
 		(pts
-			(xy 71.12 74.93) (xy 71.12 80.01)
-		)
-		(stroke
-			(width 0)
-			(type default)
-		)
-	)
-	(wire
-		(pts
-			(xy 128.27 91.44) (xy 119.38 91.44)
+			(xy 123.19 92.71) (xy 119.38 92.71)
 		)
 		(stroke
@@
 	(wire
 		(pts
+			(xy 128.27 88.9) (xy 151.13 88.9)
+		)
+		(stroke
+			(width 0)
+			(type default)
+		)
+	)
+	(wire
+		(pts
 			(xy 106.68 114.3) (xy 106.68 113.03)
-		)
-		(stroke
-			(width 0)
-			(type default)
-		)
-	)
-	(wire
-		(pts
-			(xy 54.61 80.01) (xy 54.61 90.17)
 		)
 		(stroke
@@
 			)
 		)
-		(property "Sim.Library" "BB112.cir"
+		(property "Sim.Library" "1SV149.lib"
 			(at 100.33 96.52 0)
 			(hide yes)
@@
 			)
 		)
-		(property "Sim.Name" "BB112"
+		(property "Sim.Name" "D1SV149"
 			(at 100.33 96.52 0)
 			(hide yes)
@@
 	(symbol
 		(lib_id "Connector:Conn_Coaxial")
-		(at 133.35 91.44 0)
+		(at 128.27 92.71 0)
 		(unit 1)
 		(body_style 1)
-		(exclude_from_sim no)
+		(exclude_from_sim yes)
 		(in_bom yes)
 		(on_board yes)
@@
 		(fields_autoplaced yes)
 		(property "Reference" "J3"
-			(at 137.16 90.4631 0)
+			(at 132.08 91.7331 0)
 			(show_name no)
 			(do_not_autoplace no)
@@
 		)
 		(property "Value" "Conn_Coaxial"
-			(at 137.16 93.0031 0)
+			(at 132.08 94.2731 0)
 			(show_name no)
 			(do_not_autoplace no)
@@
 		)
 		(property "Footprint" "Connector_Coaxial:BNC_Amphenol_031-5539_Vertical"
-			(at 133.35 91.44 0)
+			(at 128.27 92.71 0)
 			(hide yes)
 			(show_name no)
@@
 		)
 		(property "Datasheet" ""
-			(at 133.35 91.44 0)
+			(at 128.27 92.71 0)
 			(hide yes)
 			(show_name no)
@@
 		)
 		(property "Description" "coaxial connector (BNC, SMA, SMB, SMC, Cinch/RCA, LEMO, ...)"
-			(at 133.35 91.44 0)
+			(at 128.27 92.71 0)
 			(hide yes)
 			(show_name no)
@@
 	(symbol
 		(lib_id "Connector:Conn_Coaxial")
-		(at 54.61 74.93 90)
+		(at 128.27 73.66 0)
 		(unit 1)
 		(body_style 1)
-		(exclude_from_sim no)
+		(exclude_from_sim yes)
 		(in_bom yes)
 		(on_board yes)
@@
 		(fields_autoplaced yes)
 		(property "Reference" "J2"
-			(at 54.9032 68.58 90)
-			(show_name no)
-			(do_not_autoplace no)
-			(effects
-				(font
-					(size 1.27 1.27)
-				)
+			(at 132.08 72.6831 0)
+			(show_name no)
+			(do_not_autoplace no)
+			(effects
+				(font
+					(size 1.27 1.27)
+				)
+				(justify left)
 			)
 		)
 		(property "Value" "Conn_Coaxial"
-			(at 54.9032 71.12 90)
-			(show_name no)
-			(do_not_autoplace no)
-			(effects
-				(font
-					(size 1.27 1.27)
-				)
+			(at 132.08 75.2231 0)
+			(show_name no)
+			(do_not_autoplace no)
+			(effects
+				(font
+					(size 1.27 1.27)
+				)
+				(justify left)
 			)
 		)
 		(property "Footprint" "Connector_Coaxial:BNC_Amphenol_031-5539_Vertical"
-			(at 54.61 74.93 0)
+			(at 128.27 73.66 0)
 			(hide yes)
 			(show_name no)
@@
 		)
 		(property "Datasheet" ""
-			(at 54.61 74.93 0)
+			(at 128.27 73.66 0)
 			(hide yes)
 			(show_name no)
@@
 		)
 		(property "Description" "coaxial connector (BNC, SMA, SMB, SMC, Cinch/RCA, LEMO, ...)"
-			(at 54.61 74.93 0)
+			(at 128.27 73.66 0)
 			(hide yes)
 			(show_name no)
@@
 			)
 		)
-		(property "Sim.Library" "BB112.cir"
+		(property "Sim.Library" "1SV149.lib"
 			(at 88.9 96.52 0)
 			(hide yes)
@@
 			)
 		)
-		(property "Sim.Name" "BB112"
+		(property "Sim.Name" "D1SV149"
 			(at 88.9 96.52 0)
 			(hide yes)
@@
 			)
 		)
-		(property "Value" "500k"
+		(property "Value" "1500k"
 			(at 74.93 106.934 90)
 			(show_name no)
